File: 8x8x8/Diagrams/breaker/breaker.kicad_sch (KiCad schematic)
At the start: 1 part

Commit message: minor change
Other:
- note added: "Pinouts: 1: Common (connect to +) 4: Normally open circuit (will only allow power flow if signal given here) 2: Coil 1 (+ OR -, not sure) 5: Coil 2 (opposite of Coil 1)"
- note removed: "Pinouts: 1: Common (connect to +) 4: Normally closed (will only allow power flow if signal given here) 2: Coil 1 (+ OR -, not sure) 5: Coil 2 (opposite of Coil 1)"
Changed lines of the file:
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@@
     (effects (font (size 1.27 1.27)) (justify left bottom))
   )
-  (text "Pinouts:\n1: Common (connect to +)\n4: Normally closed (will only allow power flow if signal given here)\n2: Coil 1 (+ OR -, not sure)\n5: Coil 2 (opposite of Coil 1)\n"
+  (text "Pinouts:\n1: Common (connect to +)\n4: Normally open circuit (will only allow power flow if signal given here)\n2: Coil 1 (+ OR -, not sure)\n5: Coil 2 (opposite of Coil 1)\n"
     (at 109.22 90.17 0)
     (effects (font (size 1.27 1.27)) (justify left bottom))
@@
   (symbol_instances
     (path "/5d0be09d-133e-4cac-b0d8-fd336835cc6c"
-      (reference "K2") (unit 1) (value "SANYOU_SRD_Form_B (Normally Open)") (footprint "Relay_THT:Relay_SPST_SANYOU_SRD_Series_Form_B")
+      (reference "K2") (unit 1) (value "SANYOU_SRD_Form_B (Normally Open Relay)") (footprint "Relay_THT:Relay_SPST_SANYOU_SRD_Series_Form_B")
     )
   )
