File: 4x4x4/Diagrams/pcb/pcb.kicad_pcb (KiCad board)
At the start: 2 copper layers, 78 parts, among them J1 Conn_01x04_Female, J10 Conn_01x04_Female, J11 Conn_01x04_Female, J12 Conn_01x04_Female, J13 Conn_01x04_Female, J14 Conn_01x04_Female, J2 Conn_01x06_Female, J3 Conn_01x04_Female, J4 Conn_01x04_Female, J5 Conn_01x04_Female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

Commit message: finish general layout for pcb
Parts:
- removed R5: 10000, Resistor_THT:R_Axial_DIN0204_L3.6mm_D1.6mm_P5.08mm_Horizontal
- moved R50 127.6 mm to (98.5, 148.6), turned to 180 degrees
- moved R53 108.7 mm to (98.5, 141.0), turned to 180 degrees
- moved R46 107.8 mm to (98.5, 128.3), turned to 180 degrees
- moved R48 103.2 mm to (98.5, 123.2), turned to 180 degrees
- moved R51 103.1 mm to (98.5, 146.1), turned to 180 degrees
- moved U4 94.4 mm to (74.9, 66.0), turned to 180 degrees
- moved R47 91.9 mm to (98.5, 125.7), turned to 180 degrees
- moved J2 86.6 mm to (99.4, 154.8), turned to 180 degrees
- moved J7 85.8 mm to (65.0, 79.0), turned to 90 degrees
- moved R1 85.1 mm to (88.6, 126.7), turned to 90 degrees
- moved J8 84.8 mm to (65.0, 61.7), turned to 90 degrees
- moved R38 83.8 mm to (98.4, 92.6), turned to 180 degrees
- moved R52 83.2 mm to (98.5, 143.5), turned to 180 degrees
- moved R2 80.8 mm to (85.6, 126.7), turned to 90 degrees
- moved Q3 78.1 mm to (87.6, 116.1)
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
Commit message: layout pcb complete
Parts:
- J1, J10, J11, J12, J13, J14, J3, J4, J5, J6, J7, J8, J9: footprint Connector_Molex:Molex_Micro-Fit_3.0_43650-0400_1x04_P3.00mm_Horizontal -> TerminalBlock_Phoenix:TerminalBlock_Phoenix_MKDS-1,5-4-5.08_1x04_P5.08mm_Horizontal
- J2: footprint Connector_Molex:Molex_Micro-Fit_3.0_43650-0600_1x06_P3.00mm_Horizontal -> TerminalBlock_Phoenix:TerminalBlock_Phoenix_PT-1,5-6-5.0-H_1x06_P5.00mm_Horizontal
- moved J1 126.6 mm to (78.7, 28.2), turned to 0 degrees
- moved Q3 42.4 mm to (88.9, 73.7)
- moved Q4 42.4 mm to (82.3, 73.7)
- moved R3 39.4 mm to (86.9, 87.6)
- moved R4 39.4 mm to (83.8, 87.6)
- moved J9 21.0 mm to (108.9, 31.8)
- moved J10 16.9 mm to (108.9, 53.3)
- moved U5 16.8 mm to (96.5, 49.5)
- moved R34 16.8 mm to (101.6, 63.5)
- moved R36 16.8 mm to (101.6, 58.4)
- moved R30 16.8 mm to (101.6, 42.9)
- moved R31 16.8 mm to (101.6, 40.6)
- moved R32 16.8 mm to (101.6, 38.1)
- moved R33 16.8 mm to (101.6, 35.6)
- moved R35 16.8 mm to (101.6, 61.0)
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Connections:
- Q1 pad 1: Net-(J1-Pad4) -> Net-(J1-Pad1)
- Q2 pad 1: Net-(J1-Pad3) -> Net-(J1-Pad2)
- Q3 pad 1: Net-(J1-Pad2) -> Net-(J1-Pad3)
- Q4 pad 1: Net-(J1-Pad1) -> Net-(J1-Pad4)
- R1 pad 2: Net-(Q4-Pad2) -> Net-(Q1-Pad2)
- R2 pad 2: Net-(Q3-Pad2) -> Net-(Q2-Pad2)
- R3 pad 2: Net-(Q2-Pad2) -> Net-(Q3-Pad2)
- R4 pad 2: Net-(Q1-Pad2) -> Net-(Q4-Pad2)
Routing:
- net GND: track 0.00 -> 300.4 mm
- net Net-(J2-Pad6): track 0.00 -> 246.8 mm

Commit message: review pcb
Parts:
- moved J1 156.0 mm to (68.1, 183.9), turned to 90 degrees
- moved Q3 98.3 mm to (57.6, 166.9), turned to -90 degrees
- moved Q4 98.3 mm to (51.0, 166.9), turned to -90 degrees
- moved R3 93.0 mm to (55.6, 175.3), turned to 0 degrees
- moved R4 89.6 mm to (55.6, 172.7), turned to 0 degrees
- moved Q1 81.2 mm to (51.1, 186.2), turned to 90 degrees
- moved Q2 76.0 mm to (57.7, 186.2), turned to 90 degrees
- moved J2 65.8 mm to (40.4, 188.7), turned to 90 degrees
- moved R1 61.1 mm to (55.6, 180.3), turned to 0 degrees
- moved R2 57.4 mm to (55.6, 177.8), turned to 0 degrees
- moved U1 48.7 mm to (50.5, 176.5), turned to 90 degrees
- moved J3 31.9 mm to (34.6, 138.7)
Connections:
- J2 pad 3: Net-(J2-Pad3) -> Net-(U1-Pad13)
- U1 pad 1: Net-(R2-Pad1) -> Net-(R1-Pad1)
- U1 pad 12: Net-(J2-Pad3) -> Net-(J2-Pad4)
- U1 pad 13: Net-(J2-Pad2) -> Net-(U1-Pad13)
- U1 pad 14: Net-(J2-Pad4) -> Net-(J2-Pad2)
- U1 pad 15: Net-(R1-Pad1) -> unconnected-(U1-Pad15)
- U1 pad 2: Net-(R3-Pad1) -> Net-(R2-Pad1)
- U1 pad 3: Net-(R4-Pad1) -> Net-(R3-Pad1)
- U1 pad 4: unconnected-(U1-Pad4) -> Net-(R4-Pad1)
- U2 pad 12: Net-(J2-Pad3) -> Net-(J2-Pad4)
- U2 pad 13: Net-(J2-Pad2) -> Net-(U1-Pad13)
- U3 pad 12: Net-(J2-Pad3) -> Net-(J2-Pad4)
- U3 pad 13: Net-(J2-Pad2) -> Net-(U1-Pad13)
- U4 pad 12: Net-(J2-Pad3) -> Net-(J2-Pad4)
- U4 pad 13: Net-(J2-Pad2) -> Net-(U1-Pad13)
- U5 pad 12: Net-(J2-Pad3) -> Net-(J2-Pad4)
- U5 pad 13: Net-(J2-Pad2) -> Net-(U1-Pad13)
- U6 pad 12: Net-(J2-Pad3) -> Net-(J2-Pad4)
- U6 pad 13: Net-(J2-Pad2) -> Net-(U1-Pad13)
- U7 pad 12: Net-(J2-Pad3) -> Net-(J2-Pad4)
- U7 pad 13: Net-(J2-Pad2) -> Net-(U1-Pad13)
Routing:
- net GND: track 300.4 -> 48.2 mm
- net Net-(J2-Pad6): track 246.8 -> 22.1 mm
- net Net-(J1-Pad1): track 0.00 -> 19.3 mm
- net Net-(J1-Pad4): track 0.00 -> 19.1 mm
- net Net-(J1-Pad2): track 0.00 -> 14.0 mm
- net Net-(Q3-Pad2): track 0.00 -> 13.9 mm
- net Net-(J1-Pad3): track 0.00 -> 13.8 mm
- net Net-(Q4-Pad2): track 0.00 -> 13.6 mm
- net Net-(Q2-Pad2): track 0.00 -> 11.6 mm
- net Net-(Q1-Pad2): track 0.00 -> 10.8 mm
- net Net-(J2-Pad5): track 0.00 -> 9.81 mm
- net Net-(J2-Pad2): track 0.00 -> 9.56 mm
- net Net-(J2-Pad4): track 0.00 -> 8.27 mm
- net Net-(U1-Pad13): track 0.00 -> 8.01 mm
- net Net-(R4-Pad1): track 0.00 -> 5.39 mm
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