File: 8x8x8/Diagrams/AC_to_DC5V_Circuit/AC_to_DC5V_Circuit.kicad_sch (KiCad schematic)
At the start: 30 parts, among them J1 Conn_01x01 (Arduino Signal Pi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, J10 Conn_01x01 (Q3 +5V), J11 Conn_01x01 (Q3 -5V), J12 Conn_01x01 (Q4 +5V), J13 Conn_01x01 (Q4 -5V), J2 Conn_01x03, J3 Conn_01x01 (Arduino ground), J4 Conn_01x03, J5 Conn_01x03, J6 Conn_01x01 (Q1 +5V)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

Commit message: fix small mistake
Connections:
- net at J11.1 (Pin_1), J13.1 (Pin_1), J7.1 (Pin_1)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: no longer J5.1 (Pin_1), J5.2 (Pin_2), U1.3 (GND), U2.3 (GND), U3.3 (GND), U4.3 (GND)
- net at U4.5 (~{ON}/OFF): now also J5.1 (Pin_1), J5.2 (Pin_2), U1.3 (GND), U1.5 (~{ON}/OFF), U2.3 (GND), U2.5 (~{ON}/OFF), U3.3 (GND), U3.5 (~{ON}/OFF), U4.3 (GND)
Changed lines of the file:
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@@
   (junction (at 129.54 157.48) (diameter 0) (color 0 0 0 0)
   )
+  (junction (at 59.69 119.38) (diameter 0) (color 0 0 0 0)
+  )
   (junction (at 86.36 152.4) (diameter 0) (color 0 0 0 0)
   )
@@
   (junction (at 116.84 157.48) (diameter 0) (color 0 0 0 0)
   )
+  (junction (at 59.69 140.97) (diameter 0) (color 0 0 0 0)
+  )
   (junction (at 54.61 152.4) (diameter 0) (color 0 0 0 0)
   )
@@
   (junction (at 116.84 135.89) (diameter 0) (color 0 0 0 0)
   )
+  (junction (at 59.69 162.56) (diameter 0) (color 0 0 0 0)
+  )
   (junction (at 107.95 135.89) (diameter 0) (color 0 0 0 0)
   )
@@
   (junction (at 138.43 142.24) (diameter 0) (color 0 0 0 0)
   )
+  (junction (at 59.69 184.15) (diameter 0) (color 0 0 0 0)
+  )
   (junction (at 107.95 179.07) (diameter 0) (color 0 0 0 0)
-  )
-  (junction (at 49.53 184.15) (diameter 0) (color 0 0 0 0)
-  )
-  (junction (at 86.36 191.77) (diameter 0) (color 0 0 0 0)
   )
   (junction (at 116.84 114.3) (diameter 0) (color 0 0 0 0)
@@
     (stroke (width 0) (type default) (color 0 0 0 0))
   )
+  (wire (pts (xy 59.69 119.38) (xy 72.39 119.38))
+    (stroke (width 0) (type default) (color 0 0 0 0))
+  )
   (wire (pts (xy 86.36 109.22) (xy 86.36 130.81))
     (stroke (width 0) (type default) (color 0 0 0 0))
@@
     (stroke (width 0) (type default) (color 0 0 0 0))
   )
+  (wire (pts (xy 59.69 179.07) (xy 59.69 184.15))
+    (stroke (width 0) (type default) (color 0 0 0 0))
+  )
   (wire (pts (xy 99.06 46.99) (xy 179.07 46.99))
     (stroke (width 0) (type default) (color 0 0 0 0))
@@
     (stroke (width 0) (type default) (color 0 0 0 0))
   )
-  (wire (pts (xy 49.53 140.97) (xy 72.39 140.97))
-    (stroke (width 0) (type default) (color 0 0 0 0))
-  )
-  (wire (pts (xy 49.53 162.56) (xy 72.39 162.56))
+  (wire (pts (xy 59.69 135.89) (xy 59.69 140.97))
+    (stroke (width 0) (type default) (color 0 0 0 0))
+  )
+  (wire (pts (xy 49.53 140.97) (xy 59.69 140.97))
+    (stroke (width 0) (type default) (color 0 0 0 0))
+  )
+  (wire (pts (xy 49.53 162.56) (xy 59.69 162.56))
     (stroke (width 0) (type default) (color 0 0 0 0))
   )
@@
     (stroke (width 0) (type default) (color 0 0 0 0))
   )
+  (wire (pts (xy 59.69 162.56) (xy 72.39 162.56))
+    (stroke (width 0) (type default) (color 0 0 0 0))
+  )
   (wire (pts (xy 168.91 77.47) (xy 168.91 52.07))
     (stroke (width 0) (type default) (color 0 0 0 0))
@@
     (stroke (width 0) (type default) (color 0 0 0 0))
   )
-  (wire (pts (xy 49.53 119.38) (xy 72.39 119.38))
-    (stroke (width 0) (type default) (color 0 0 0 0))
-  )
-  (wire (pts (xy 49.53 184.15) (xy 72.39 184.15))
+  (wire (pts (xy 49.53 119.38) (xy 59.69 119.38))
+    (stroke (width 0) (type default) (color 0 0 0 0))
+  )
+  (wire (pts (xy 49.53 184.15) (xy 59.69 184.15))
     (stroke (width 0) (type default) (color 0 0 0 0))
   )
@@
     (stroke (width 0) (type default) (color 0 0 0 0))
   )
+  (wire (pts (xy 59.69 184.15) (xy 72.39 184.15))
+    (stroke (width 0) (type default) (color 0 0 0 0))
+  )
   (wire (pts (xy 97.79 187.96) (xy 95.25 187.96))
     (stroke (width 0) (type default) (color 0 0 0 0))
@@
     (stroke (width 0) (type default) (color 0 0 0 0))
   )
+  (wire (pts (xy 59.69 157.48) (xy 59.69 162.56))
+    (stroke (width 0) (type default) (color 0 0 0 0))
+  )
   (polyline (pts (xy 19.05 27.94) (xy 172.72 27.94))
     (stroke (width 0) (type default) (color 0 0 0 0))
@@
     (stroke (width 0) (type default) (color 0 0 0 0))
   )
-  (wire (pts (xy 49.53 191.77) (xy 86.36 191.77))
+  (wire (pts (xy 59.69 140.97) (xy 72.39 140.97))
     (stroke (width 0) (type default) (color 0 0 0 0))
   )
@@
     (stroke (width 0) (type default) (color 0 0 0 0))
   )
+  (wire (pts (xy 59.69 114.3) (xy 59.69 119.38))
+    (stroke (width 0) (type default) (color 0 0 0 0))
+  )
   (wire (pts (xy 57.15 62.23) (xy 88.9 62.23))
     (stroke (width 0) (type default) (color 0 0 0 0))
@@
     (stroke (width 0) (type default) (color 0 0 0 0))
   )
-  (wire (pts (xy 49.53 184.15) (xy 49.53 191.77))
-    (stroke (width 0) (type default) (color 0 0 0 0))
-  )

Commit message: small correction to dc-
Parts:
- removed J5: Conn_01x03, TerminalBlock_Phoenix:TerminalBlock_Phoenix_MKDS-1,5-3_1x03_P5.00mm_Horizontal, symbol Connector_Generic:Conn_01x03
- added J5: (no value), symbol Connector_Generic:Conn_01x02
Connections:
- net at U1.3 (GND), U1.5 (~{ON}/OFF), U2.3 (GND)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: now also J5.1 (Pin_1)
- net at U1.1 (VIN), U2.1 (VIN), U3.1 (VIN)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: now also J5.2 (Pin_2)
Other:
- note added: "1.1.0"
- note added: "Pinouts: 1: DC+ 2: GND 12V, 5A"
- note removed: "1.0.0"
- note removed: "3"
- note removed: "Can you connect -12VDC to GND?!?"
- note removed: "Pinouts: 1: DC+ 2: DC- 3: GND 12V, 5A"
- note removed: "o"
- moved on the sheet: J9
Changed lines of the file:
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@@
   (junction (at 107.95 135.89) (diameter 0) (color 0 0 0 0)
   )
-  (junction (at 49.53 114.3) (diameter 0) (color 0 0 0 0)
-  )
   (junction (at 95.25 135.89) (diameter 0) (color 0 0 0 0)
   )
   (junction (at 49.53 140.97) (diameter 0) (color 0 0 0 0)
   )
-  (junction (at 138.43 142.24) (diameter 0) (color 0 0 0 0)
-  )
   (junction (at 59.69 184.15) (diameter 0) (color 0 0 0 0)
   )
@@
   )
   (junction (at 95.25 157.48) (diameter 0) (color 0 0 0 0)
+  )
+  (junction (at 138.43 140.97) (diameter 0) (color 0 0 0 0)
   )
   (no_connect (at 138.43 179.07))
@@
     (stroke (width 0) (type default) (color 0 0 0 0))
   )
-  (wire (pts (xy 27.94 97.79) (xy 265.43 97.79))
-    (stroke (width 0) (type default) (color 0 0 0 0))
-  )
   (wire (pts (xy 25.4 95.25) (xy 262.89 95.25))
     (stroke (width 0) (type default) (color 0 0 0 0))
@@
     (stroke (width 0) (type default) (color 0 0 0 0))
   )
-  (polyline (pts (xy 173.99 93.98) (xy 173.99 196.85))
+  (polyline (pts (xy 172.72 93.98) (xy 172.72 196.85))
     (stroke (width 0) (type default) (color 0 0 0 0))
   )
@@
     (stroke (width 0) (type default) (color 0 0 0 0))
   )
-  (wire (pts (xy 50.8 114.3) (xy 49.53 114.3))
-    (stroke (width 0) (type default) (color 0 0 0 0))
-  )
   (wire (pts (xy 95.25 144.78) (xy 97.79 144.78))
     (stroke (width 0) (type default) (color 0 0 0 0))
@@
     (stroke (width 0) (type default) (color 0 0 0 0))
   )
+  (wire (pts (xy 138.43 140.97) (xy 138.43 162.56))
+    (stroke (width 0) (type default) (color 0 0 0 0))
+  )
   (wire (pts (xy 129.54 123.19) (xy 129.54 114.3))
     (stroke (width 0) (type default) (color 0 0 0 0))
@@
     (stroke (width 0) (type default) (color 0 0 0 0))
   )
+  (wire (pts (xy 138.43 140.97) (xy 142.24 140.97))
+    (stroke (width 0) (type default) (color 0 0 0 0))
+  )
   (wire (pts (xy 49.53 140.97) (xy 59.69 140.97))
     (stroke (width 0) (type default) (color 0 0 0 0))
@@
     (stroke (width 0) (type default) (color 0 0 0 0))
   )
-  (polyline (pts (xy 19.05 93.98) (xy 173.99 93.98))
+  (polyline (pts (xy 19.05 93.98) (xy 172.72 93.98))
     (stroke (width 0) (type default) (color 0 0 0 0))
   )
@@
     (stroke (width 0) (type default) (color 0 0 0 0))
   )
-  (polyline (pts (xy 173.99 196.85) (xy 15.24 196.85))
+  (polyline (pts (xy 172.72 196.85) (xy 15.24 196.85))
     (stroke (width 0) (type default) (color 0 0 0 0))
   )
@@
     (stroke (width 0) (type default) (color 0 0 0 0))
   )
-  (wire (pts (xy 265.43 52.07) (xy 265.43 97.79))
-    (stroke (width 0) (type default) (color 0 0 0 0))
-  )
   (wire (pts (xy 129.54 157.48) (xy 129.54 166.37))
     (stroke (width 0) (type default) (color 0 0 0 0))
@@
     (stroke (width 0) (type default) (color 0 0 0 0))
   )
-  (wire (pts (xy 50.8 111.76) (xy 50.8 114.3))
-    (stroke (width 0) (type default) (color 0 0 0 0))
-  )
   (wire (pts (xy 95.25 187.96) (xy 95.25 179.07))
     (stroke (width 0) (type default) (color 0 0 0 0))
@@
     (stroke (width 0) (type default) (color 0 0 0 0))
   )
-  (wire (pts (xy 138.43 142.24) (xy 142.24 142.24))
-    (stroke (width 0) (type default) (color 0 0 0 0))
-  )
   (wire (pts (xy 127 114.3) (xy 129.54 114.3))
     (stroke (width 0) (type default) (color 0 0 0 0))
@@
     (stroke (width 0) (type default) (color 0 0 0 0))
   )
-  (wire (pts (xy 138.43 142.24) (xy 138.43 162.56))
+  (wire (pts (xy 138.43 119.38) (xy 138.43 140.97))
     (stroke (width 0) (type default) (color 0 0 0 0))
   )
@@
     (stroke (width 0) (type default) (color 0 0 0 0))
   )
+  (wire (pts (xy 259.08 49.53) (xy 259.08 50.8))
+    (stroke (width 0) (type default) (color 0 0 0 0))
+  )
   (polyline (pts (xy 19.05 27.94) (xy 172.72 27.94))
     (stroke (width 0) (type default) (color 0 0 0 0))
@@
     (stroke (width 0) (type default) (color 0 0 0 0))
   )
-  (wire (pts (xy 259.08 52.07) (xy 265.43 52.07))
-    (stroke (width 0) (type default) (color 0 0 0 0))
-  )
   (wire (pts (xy 129.54 157.48) (xy 142.24 157.48))
     (stroke (width 0) (type default) (color 0 0 0 0))
@@
     (stroke (width 0) (type default) (color 0 0 0 0))
   )
-  (wire (pts (xy 27.94 111.76) (xy 50.8 111.76))
-    (stroke (width 0) (type default) (color 0 0 0 0))
-  )
   (wire (pts (xy 138.43 184.15) (xy 138.43 191.77))
     (stroke (width 0) (type default) (color 0 0 0 0))
@@
     (stroke (width 0) (type default) (color 0 0 0 0))
   )
+  (wire (pts (xy 259.08 53.34) (xy 259.08 54.61))
+    (stroke (width 0) (type default) (color 0 0 0 0))
+  )
   (polyline (pts (xy 172.72 27.94) (xy 172.72 90.17))
     (stroke (width 0) (type default) (color 0 0 0 0))
@@
     (stroke (width 0) (type default) (color 0 0 0 0))
   )
-  (wire (pts (xy 138.43 119.38) (xy 138.43 142.24))
-    (stroke (width 0) (type default) (color 0 0 0 0))
-  )
   (wire (pts (xy 107.95 135.89) (xy 107.95 144.78))
     (stroke (width 0) (type default) (color 0 0 0 0))
@@
   )
   (wire (pts (xy 59.69 140.97) (xy 72.39 140.97))
-    (stroke (width 0) (type default) (color 0 0 0 0))
-  )
-  (wire (pts (xy 27.94 97.79) (xy 27.94 111.76))
     (stroke (width 0) (type default) (color 0 0 0 0))
   )
@@
     (effects (font (size 1.27 1.27)) (justify left bottom))
   )
-  (text "1.0.0" (at 269.24 194.31 0)
+  (text "1.1.0" (at 269.24 194.31 0)
     (effects (font (size 1.27 1.27)) (justify left bottom))
   )
@@
     (effects (font (size 1.27 1.27)) (justify left bottom))
   )
-  (text "2" (at 30.48 111.76 0)
+  (text "2" (at 30.48 114.3 0)
     (effects (font (size 1.27 1.27)) (justify left bottom))
   )
-  (text "Pinouts:\n1: DC+\n2: DC-\n3: GND\n\n12V, 5A" (at 21.59 133.35 0)
+  (text "Pinouts:\n1: DC+\n2: GND\n\n12V, 5A" (at 21.59 133.35 0)
     (effects (font (size 1.27 1.27)) (justify left bottom))
   )
-  (text "12VDC to 5VDC\nBuck Convertor" (at 179.07 149.86 0)
+  (text "12VDC to 5VDC\nBuck Convertor" (at 175.26 149.86 0)
     (effects (font (size 6.35 6.35)) (justify left bottom))
-  )
-  (text "Can you connect\n-12VDC to GND?!?" (at 30.48 119.38 0)
-    (effects (font (size 1.27 1.27)) (justify left bottom))
   )
   (text "AC to DC Converter" (at 173.99 26.67 0)
@@
     (effects (font (size 1.27 1.27)) (justify left bottom))
   )
-  (text "o" (at 45.72 120.65 0)
-    (effects (font (size 10 10)) (justify left bottom))
-  )
-  (text "3" (at 30.48 114.3 0)
-    (effects (font (size 1.27 1.27)) (justify left bottom))
-  )
   (text "AC Relay Breaker" (at 50.8 25.4 0)
     (effects (font (size 6.35 6.35)) (justify left bottom))
   )
-  (text "- Alternative buck converter is the LM2575-5.0BT (breadboard-friendly)"
+  (text "- Alternative buck converter is the \n  LM2575-5.0BT (breadboard-friendly)"
     (at 16.51 195.58 0)
     (effects (font (size 1.27 1.27)) (justify left bottom))
@@
     (pin "1")
   )
-  (symbol (lib_id "Connector_Generic:Conn_01x03") (at 254 52.07 180) (unit 1)
-    (in_bom yes) (on_board yes) (fields_autoplaced)
-    (property "Reference" "J5" (id 0) (at 254 43.18 0))
-    (property "Value" "Conn_01x03" (id 1) (at 254 45.72 0))
-    (property "Footprint" "TerminalBlock_Phoenix:TerminalBlock_Phoenix_MKDS-1,5-3_1x03_P5.00mm_Horizontal" (id 2) (at 254 52.07 0)
-      (effects (font (size 1.27 1.27)) hide)
-    )
-    (property "Datasheet" "~" (id 3) (at 254 52.07 0)
-      (effects (font (size 1.27 1.27)) hide)
-    )
-    (pin "1")
-    (pin "2")
-    (pin "3")
-  )
   (symbol (lib_id "Diode:1N4007") (at 101.6 187.96 0) (unit 1)
     (in_bom yes) (on_board yes) (fields_autoplaced)
@@
     (pin "2")
   )
+  (symbol (lib_id "Connector_Generic:Conn_01x02") (at 254 53.34 180) (unit 1)
+    (in_bom yes) (on_board yes) (fields_autoplaced)
+    (property "Reference" "J5" (id 0) (at 254 44.45 0))
+    (property "Value" "" (id 1) (at 254 46.99 0))
+    (property "Footprint" "" (id 2) (at 254 53.34 0)
+      (effects (font (size 1.27 1.27)) hide)
+    )
+    (property "Datasheet" "~" (id 3) (at 254 53.34 0)
+      (effects (font (size 1.27 1.27)) hide)
+    )
+    (pin "1")
+    (pin "2")
+  )
   (symbol (lib_id "Connector_Generic:Conn_01x01") (at 147.32 119.38 0) (unit 1)
     (in_bom yes) (on_board yes) (fields_autoplaced)
@@
     (pin "2")
   )
-  (symbol (lib_id "Connector_Generic:Conn_01x01") (at 147.32 142.24 0) (unit 1)
-    (in_bom yes) (on_board yes) (fields_autoplaced)
-    (property "Reference" "J9" (id 0) (at 149.86 140.9699 0)
-      (effects (font (size 1.27 1.27)) (justify left))
-    )
-    (property "Value" "Conn_01x01 (Q2 -5V)" (id 1) (at 149.86 143.5099 0)
-      (effects (font (size 1.27 1.27)) (justify left))
-    )
-    (property "Footprint" "Connector_Wire:SolderWirePad_1x01_SMD_1x2mm" (id 2) (at 147.32 142.24 0)
-      (effects (font (size 1.27 1.27)) hide)
-    )
-    (property "Datasheet" "~" (id 3) (at 147.32 142.24 0)
+  (symbol (lib_id "Connector_Generic:Conn_01x01") (at 147.32 140.97 0) (unit 1)
+    (in_bom yes) (on_board yes) (fields_autoplaced)
+    (property "Reference" "J9" (id 0) (at 149.86 139.6999 0)
+      (effects (font (size 1.27 1.27)) (justify left))
+    )
+    (property "Value" "Conn_01x01 (Q2 -5V)" (id 1) (at 149.86 142.2399 0)
+      (effects (font (size 1.27 1.27)) (justify left))
+    )
+    (property "Footprint" "Connector_Wire:SolderWirePad_1x01_SMD_1x2mm" (id 2) (at 147.32 140.97 0)
+      (effects (font (size 1.27 1.27)) hide)
+    )
+    (property "Datasheet" "~" (id 3) (at 147.32 140.97 0)
       (effects (font (size 1.27 1.27)) hide)
     )
@@
       (reference "J4") (unit 1) (value "Conn_01x03") (footprint "TerminalBlock_Phoenix:TerminalBlock_Phoenix_MKDS-1,5-3_1x03_P5.00mm_Horizontal")
     )
-    (path "/4d9738f4-4bc6-4c31-8234-e35461a8bea5"
-      (reference "J5") (unit 1) (value "Conn_01x03") (footprint "TerminalBlock_Phoenix:TerminalBlock_Phoenix_MKDS-1,5-3_1x03_P5.00mm_Horizontal")
+    (path "/5221a8e0-f9f5-4fec-b777-d81fe5a4a4c5"
+      (reference "J5") (unit 1) (value "Conn_01x02") (footprint "TerminalBlock_Phoenix:TerminalBlock_Phoenix_MKDS-1,5-2_1x02_P5.00mm_Horizontal")
     )
     (path "/716fbf8b-610f-458f-aeb1-927a792e8911"

Commit message: add notes
Parts:
- J5: value (none) -> Conn_01x02; footprint (none) -> TerminalBlock_Phoenix:TerminalBlock_Phoenix_MKDS-1,5-2_1x02_P5.00mm_Horizontal
Other:
- note added: "add resistor to make output 600mA max for 2N2222A transistor"
- note added: "fix capacitor labelling"
Changed lines of the file:
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@@
     (stroke (width 0) (type default) (color 0 0 0 0))
+  )
+  (text "add resistor to make output 600mA max for 2N2222A transistor"
+    (at 144.78 125.73 0)
+    (effects (font (size 1.27 1.27)) (justify left bottom))
   )
   (text "June 30 2022" (at 207.01 194.31 0)
@@
   )
   (text "2" (at 30.48 114.3 0)
+    (effects (font (size 1.27 1.27)) (justify left bottom))
+  )
+  (text "fix capacitor labelling" (at 128.27 107.95 0)
     (effects (font (size 1.27 1.27)) (justify left bottom))
   )
@@
     (in_bom yes) (on_board yes) (fields_autoplaced)
     (property "Reference" "J5" (id 0) (at 254 44.45 0))
-    (property "Value" "" (id 1) (at 254 46.99 0))
-    (property "Footprint" "" (id 2) (at 254 53.34 0)
+    (property "Value" "Conn_01x02" (id 1) (at 254 46.99 0))
+    (property "Footprint" "TerminalBlock_Phoenix:TerminalBlock_Phoenix_MKDS-1,5-2_1x02_P5.00mm_Horizontal" (id 2) (at 254 53.34 0)
       (effects (font (size 1.27 1.27)) hide)
     )

Commit message: initial sketch finished
Other:
- note added: "Pinouts: 1: Common (connect to AC+) 4: Normally open circuit (will give AC+ when Coil 1+2 are active) 2: Coil 1 (DC-) 5: Coil 2 (DC+)"
- note removed: "Pinouts: 1: Common (connect to AC+) 4: Normally open circuit (will give AC- when Coil 1+2 are active) 2: Coil 1 (DC-) 5: Coil 2 (DC+)"
Changed lines of the file:
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@@
     (effects (font (size 1.27 1.27)) (justify left bottom))
   )
-  (text "Pinouts:\n1: Common (connect to AC+)\n4: Normally open circuit (will give AC- when Coil 1+2 are active)\n2: Coil 1 (DC-)\n5: Coil 2 (DC+)\n"
+  (text "Pinouts:\n1: Common (connect to AC+)\n4: Normally open circuit (will give AC+ when Coil 1+2 are active)\n2: Coil 1 (DC-)\n5: Coil 2 (DC+)\n"
     (at 102.87 68.58 0)
     (effects (font (size 1.27 1.27)) (justify left bottom))
