File: 8x8x8/Diagrams/Quad 1/Quad 1.kicad_sch (KiCad schematic)
At the start: 87 parts, among them J0 Conn_01x06_Female, J1 Conn_01x08_Female, J10 Conn_01x04_Female, J11 Conn_01x04_Female, J12 Conn_01x04_Female, J13 Conn_01x04_Female, J14 Conn_01x04_Female, J2 Conn_01x04_Female, J3 Conn_01x04_Female, J4 Conn_01x04_Female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

Commit message: update
Parts:
- removed R8: 10000, symbol Device:R
Other:
- note added: "0.3.1"
- note added: "To next Quadrant"
- note removed: "0.3.0"
- note removed: "Quad 1 to Quad 2"
Changed lines of the file:
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@@
   (junction (at 139.7 156.21) (diameter 0) (color 0 0 0 0)
   )
-  (junction (at 48.26 189.23) (diameter 0) (color 0 0 0 0)
-  )
   (junction (at 213.36 153.67) (diameter 0) (color 0 0 0 0)
   )
@@
     (stroke (width 0) (type default) (color 0 0 0 0))
   )
-  (wire (pts (xy 279.4 147.32) (xy 279.4 148.59))
-    (stroke (width 0) (type default) (color 0 0 0 0))
-  )
   (wire (pts (xy 209.55 157.48) (xy 209.55 129.54))
     (stroke (width 0) (type default) (color 0 0 0 0))
@@
     (stroke (width 0) (type default) (color 0 0 0 0))
   )
-  (wire (pts (xy 48.26 189.23) (xy 53.34 189.23))
-    (stroke (width 0) (type default) (color 0 0 0 0))
-  )
   (wire (pts (xy 247.65 137.16) (xy 248.92 137.16))
     (stroke (width 0) (type default) (color 0 0 0 0))
@@
     (stroke (width 0) (type default) (color 0 0 0 0))
   )
+  (wire (pts (xy 269.24 148.59) (xy 269.24 147.32))
+    (stroke (width 0) (type default) (color 0 0 0 0))
+  )
   (wire (pts (xy 135.89 64.77) (xy 127 64.77))
     (stroke (width 0) (type default) (color 0 0 0 0))
@@
     (stroke (width 0) (type default) (color 0 0 0 0))
   )
-  (wire (pts (xy 60.96 186.69) (xy 60.96 189.23))
-    (stroke (width 0) (type default) (color 0 0 0 0))
-  )
   (wire (pts (xy 238.76 134.62) (xy 233.68 134.62))
     (stroke (width 0) (type default) (color 0 0 0 0))
@@
     (stroke (width 0) (type default) (color 0 0 0 0))
   )
-  (wire (pts (xy 269.24 147.32) (xy 279.4 147.32))
+  (wire (pts (xy 269.24 148.59) (xy 279.4 148.59))
     (stroke (width 0) (type default) (color 0 0 0 0))
   )
@@
     (effects (font (size 1.27 1.27)) (justify left bottom))
   )
-  (text "Quad 1 to Quad 2" (at 266.7 161.29 0)
+  (text "To next Quadrant" (at 266.7 161.29 0)
     (effects (font (size 1.27 1.27)) (justify left bottom))
   )
@@
     (effects (font (size 1.27 1.27)) (justify left bottom))
   )
-  (text "0.3.0" (at 267.97 194.31 0)
+  (text "0.3.1" (at 267.97 194.31 0)
     (effects (font (size 1.27 1.27)) (justify left bottom))
   )
@@
     (pin "9")
   )
-  (symbol (lib_id "power:VCC") (at 60.96 186.69 0) (unit 1)
-    (in_bom yes) (on_board yes) (fields_autoplaced)
-    (property "Reference" "#PWR03" (id 0) (at 60.96 190.5 0)
-      (effects (font (size 1.27 1.27)) hide)
-    )
-    (property "Value" "VCC" (id 1) (at 63.5 185.4199 0)
-      (effects (font (size 1.27 1.27)) (justify left))
-    )
-    (property "Footprint" "" (id 2) (at 60.96 186.69 0)
-      (effects (font (size 1.27 1.27)) hide)
-    )
-    (property "Datasheet" "" (id 3) (at 60.96 186.69 0)
-      (effects (font (size 1.27 1.27)) hide)
-    )
-    (pin "1")
-  )
   (symbol (lib_id "74xx:74HC595") (at 259.08 134.62 0) (unit 1)
     (in_bom yes) (on_board yes) (fields_autoplaced)
@@
     (pin "2")
   )
-  (symbol (lib_id "Device:R") (at 57.15 189.23 270) (unit 1)
-    (in_bom yes) (on_board yes)
-    (property "Reference" "R8" (id 0) (at 58.42 190.5 0)
-      (effects (font (size 1.27 1.27)) (justify left))
-    )
-    (property "Value" "10000" (id 1) (at 55.88 190.5 0)
-      (effects (font (size 1.27 1.27)) (justify left))
-    )
-    (property "Footprint" "" (id 2) (at 57.15 187.452 90)
-      (effects (font (size 1.27 1.27)) hide)
-    )
-    (property "Datasheet" "~" (id 3) (at 57.15 189.23 0)
-      (effects (font (size 1.27 1.27)) hide)
-    )
-    (pin "1")
-    (pin "2")
-  )
   (symbol (lib_id "Device:R") (at 194.31 97.79 90) (unit 1)
     (in_bom yes) (on_board yes)
@@
       (reference "#PWR02") (unit 1) (value "VCC") (footprint "")
     )
-    (path "/7288ce3d-ad6e-43f5-96ca-99065d7798d0"
-      (reference "#PWR03") (unit 1) (value "VCC") (footprint "")
-    )
     (path "/eab7c737-4450-406f-9f80-b2e18bb45dd6"
       (reference "J0") (unit 1) (value "Conn_01x06_Female") (footprint "")
@@
       (reference "R7") (unit 1) (value "1000") (footprint "")
     )
-    (path "/a560f403-c7e0-4d97-9b6c-c5351bebb237"
-      (reference "R8") (unit 1) (value "10000") (footprint "")
-    )
     (path "/d547ab08-9a5d-4bc3-bdc6-eb70399817c6"
